File: pcb/pcb.kicad_sch (KiCad schematic)
At the start: 65 parts, among them J1 AudioJack4, J2 USB_C_Receptacle_USB2.0, SW1 Switch, SW10 Switch, SW11 Switch, SW12 Switch, SW13 Switch, SW14 Switch, SW15 Switch, SW16 Switch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

Commit message: new pcb
Parts:
- removed J1: AudioJack4, zzkeeb:Connector_TRRS-reversible, symbol Connector:AudioJack4
- removed J2: USB_C_Receptacle_USB2.0, zzkeeb:Connector_USB-C-mid-mount-ali-reversible-data, symbol Connector:USB_C_Receptacle_USB2.0
- removed LED1, LED10, LED11, LED12, LED13, LED14, LED15, LED16, LED17, LED18, LED2, LED3, LED4, LED5, LED6, LED7, LED8, LED9: LED_SK6812MINI-E, zzkeeb:LED_SK6812-MINI-E-reversible, symbol zzkeeb:LED_SK6812MINI-E
- removed SW15, SW16: Switch, zzkeeb:Switch_ChocV1-hotswap-reversible, symbol zzkeeb:Switch
- removed U3: RollerEncoder_EVQWGD001, zzkeeb:RotaryEncoder_EVQWGD001, symbol zzkeeb:RollerEncoder_EVQWGD001
- added FiveWay1: 5Way-Tactile_K1-1506DN-01, zzkeeb:Button_5way, symbol fingerpunch:5Way-Tactile_K1-1506DN-01
- added J1, J4: R3, Connector_PinHeader_2.54mm:PinHeader_1x01_P2.54mm_Vertical, symbol Connector:Conn_01x01_Socket
- added J3: C0, Connector_PinHeader_2.54mm:PinHeader_1x01_P2.54mm_Vertical, symbol Connector:Conn_01x01_Socket
- added J5: C2, Connector_PinHeader_2.54mm:PinHeader_1x01_P2.54mm_Vertical, symbol Connector:Conn_01x01_Socket
- added R1, R2: 4.7k, Resistor_SMD:R_1206_3216Metric_Pad1.30x1.75mm_HandSolder, symbol Device:R_Small
- added USB1 (x2): Connector_HRO-TYPE-C-31-M-12, zzkeeb:Connector_HRO-TYPE-C-31-M-12-data, symbol zzkeeb:Connector_HRO-TYPE-C-31-M-12
- D1, D10, D11, D12, D13, D14, D15, D16, D17, D18, D19, D2, D3, D4, D5, D6, D7, D8, D9: footprint zzkeeb:Diode_1N4148-SOD123-reversible-flip3d -> zzkeeb:Diode_1N4148-SOD123-no-label-reversible-flip3d
- SW1, SW10, SW11, SW12, SW13, SW14, SW2, SW3, SW4, SW5, SW6, SW7, SW8, SW9: footprint zzkeeb:Switch_ChocV1-hotswap-reversible -> zzkeeb:Switch_MX-hotswap-miny-reversible
- SW17, SW18: footprint zzkeeb:Switch_ChocV1-hotswap-reversible -> zzkeeb:Switch_KS-miny-reversible-hotswap-south
Connections:
- net GND: now also R2.1, USB1.1 (GND), USB1.1 (GND), USB1.12 (GND), USB1.12 (GND)
- net RX: now also USB1.5 (DN2), USB1.5 (DN2), USB1.7 (DN1), USB1.7 (DN1)
- net TX: now also USB1.6 (DP1), USB1.6 (DP1), USB1.8 (DP2), USB1.8 (DP2)
- net VCC: now also R1.1, USB1.11 (VBUS), USB1.11 (VBUS), USB1.2 (VBUS), USB1.2 (VBUS)
- net col0: now also FiveWay1.6, J3.1 (Pin_1)
- net col1: now also FiveWay1.1
- net col2: now also FiveWay1.3, J5.1 (Pin_1)
- net col3: now also FiveWay1.2
- net col4: now also FiveWay1.5
- net at D17.2 (A): now also J4.1 (Pin_1)
- net hand: now reaches U1.3 (2)
- net hand: now also U2.3 (2), R1.2, R2.2
- net row4: now reaches U1.6 (5)
- net row4: now also U2.18 (27), FiveWay1.4
- net at D15.2 (A): now also J1.1 (Pin_1)
- net LED: no longer names the net of U1.19 (28)
- net LED: no longer U2.19 (28)
- no-connect marks 21 -> 22
